Commit message: fix(openarm_description): point openarm_hand collision meshes at the right package
Problem
K4: with ee_type:=openarm_hand the palm (hand) collision mesh of both arms
was package://openarm_descriptions/meshes/ee/openarm_hand/collision/hand.stl.
No package of that name exists, so the collision geometry never loaded.
The visual mesh is fine, which is why RViz looked right, but MoveIt
collision checking and simulators lost the palm.

Root cause
urdf/ee/openarm_hand_macro.xacro:36 had an extra "s" after
${description_pkg}; the visual mesh on line 30 is correct.

Change
- Drop the extra "s". meshes/ee/openarm_hand/collision/hand.stl was already
  imported.
- test/urdf_checks.py: K4 removed from the known list, so M1 now blocks
  this kind of error.
- test/golden.json regenerated: only the URDF hash of the 6 openarm_hand
  combinations changes, the ros2_control summaries are untouched.

Behavior change
The openarm_hand palms (left and right) now have collision geometry. The
rendered URDF differs from before in exactly two lines (left/right hand
collision mesh filename). ros2_control unchanged, so neither real hardware
nor fake behaves differently. Same on Humble and Jazzy.

Test
Before the fix (K4 no longer known, xacro unchanged): urdf_checks 148
passed, 6 failed - M1 missing mesh .../openarm_descriptions/.../hand.stl on
all 6 openarm_hand combinations. After the xacro fix and before the golden
update: M1 passes, G1 fails on the same 6 with "URDF differs from golden
(ros2_control summary unchanged)", as intended; the golden diff is 6
sha256 lines.
Full test after the fix: linters at baseline; D1/D2 PASS; urdf_checks 154
passed, 0 failed, 18 known (K1 13, K3 1, K5 4); fake_smoke both cases
PASS. FULL TEST PASSED.

Docs: openarm_description/docs/03-openarm-hand-collision-path.md

Co-Authored-By: Claude Opus 5.5 <noreply@anthropic.com>

File: openarm_description/urdf/ee/openarm_hand_macro.xacro (robot description, xacro)
@@ -31,5 +31,5 @@
         <xacro:openarm-ee-kinematics-link config="${ee_kinematics_link}" name="${name}" />
         <geometry>
-          <mesh filename="package://${description_pkg}s/meshes/ee/${ee_type}/collision/${name}.stl" scale="0.001 0.001 0.001" />
+          <mesh filename="package://${description_pkg}/meshes/ee/${ee_type}/collision/${name}.stl" scale="0.001 0.001 0.001" />
         </geometry>
       </collision>
