Commit message: fix(openarm_description): mark real-hardware O6 dip joints mimic="false"
Problem
K3: openarm_o6_bimanual.launch.py use_fake_hardware:=false on Jazzy aborts
while ros2_control_node parses the URDF, before any plugin is loaded:
  what():  Joint 'L_thumb_dip' has mimic attribute not set to false:
           Activated mimic joints cannot have command interfaces.
So real O6 bimanual could not start on u24 with this description.

Root cause
The ten O6 *_dip joints are URDF <mimic> joints; in real-hardware mode the
ros2_control block declares them through configure_joint with
position/velocity/effort command interfaces. Jazzy rejects command
interfaces on a mimic joint unless it is marked mimic="false"; Humble has
no such check. Real mode cannot simply go state-only like fake mode:
OpenArm_v10HW exports these command interfaces and computes the dip
positions itself (openarm_ros2 c47a870 v10_simple_hardware.cpp:170-174,
:1397-1401), and how Jazzy's ResourceManager treats exported interfaces
the URDF does not declare is unverified.

Change (option chosen by the user)
- openarm.bimanual.ros2_control.xacro: the real-hardware branch of
  configure_mimic_joint writes the joint directly with the same interfaces
  and initial values as configure_joint, plus mimic="false", so
  ros2_control leaves the joint to the hardware. xacro:attribute inside
  xacro:if is silently dropped (xacro 2.1.1), hence the explicit joint;
  G1's per-joint interface summary catches any copy mistake.
- test/urdf_checks.py: F3 now gates real-hardware mode too (K3 no longer
  known).
- test/fake_smoke.py: new H1 case real_o6_parse_probe. With openarm_hardware
  NOT installed it launches openarm_o6_bimanual.launch.py
  use_fake_hardware:=false and requires the launch to stop at loading
  openarm_hardware/OpenArm_v10HW rather than at the mimic error. If
  openarm_hardware is installed, H1 is skipped and real hardware is never
  started.
- test/golden.json regenerated; only bimanual:=true ee_type:=o6
  use_fake_hardware:=false changes: the 10 dip joints gain mimic=false,
  interfaces identical (the block is keyed by content hash, so the file
  diff replaces the whole block).

Behavior change
- Jazzy: the real O6 URDF now passes ros2_control parsing and proceeds to
  load OpenArm_v10HW.
- Humble: its parser does not read the attribute, so no change (inferred;
  Humble is verified in a later batch).
- Real dip joints keep their command interfaces, still driven/reported by
  OpenArm_v10HW; hand controllers only command the 6 active joints.
- Fake mode unchanged.
- Needs on-robot validation on u24 with O6 hands.

Test
Before the fix (F3/H1 added, xacro unchanged): urdf_checks 154 passed,
1 failed (F3 on the real bimanual o6 case); H1 FAIL "ros2_control rejected
the URDF: Activated mimic joints cannot have command interfaces".
After: urdf_checks 155 passed, 0 failed, 17 known (K1 13, K5 4); fake_smoke
bimanual_openarm_hand S1-S3 PASS (gripper SKIP), bimanual_o6 S1-S4 PASS,
real_o6_parse_probe H1 PASS (LibraryLoadException for
openarm_hardware/OpenArm_v10HW, not installed); linters and D1/D2 as
before. FULL TEST PASSED.

Docs: openarm_description/docs/04-o6-mimic-real-hardware.md

Co-Authored-By: Claude Opus 5.5 <noreply@anthropic.com>

File: openarm_description/urdf/ros2_control/openarm.bimanual.ros2_control.xacro (robot description, xacro)
@@ -50,6 +50,7 @@
       <!-- O6 *_dip joints are <mimic> joints in the URDF. Jazzy refuses command interfaces
            on an active mimic joint, and the mock computes it from the URDF <mimic> anyway,
-           so in fake mode it only gets state interfaces. Real hardware keeps the full set:
-           OpenArm_v10HW exports and drives these joints itself. -->
+           so in fake mode it only gets state interfaces. Real hardware keeps the full set
+           (same as configure_joint) and is marked mimic="false": OpenArm_v10HW exports and
+           drives these joints itself. Humble ignores the attribute. -->
       <xacro:macro name="configure_mimic_joint" params="joint_name initial_position">
         <xacro:if value="${use_fake_hardware}">
@@ -67,5 +68,18 @@
         </xacro:if>
         <xacro:unless value="${use_fake_hardware}">
-          <xacro:configure_joint joint_name="${joint_name}" initial_position="${initial_position}"/>
+          <joint name="${joint_name}" mimic="false">
+            <command_interface name="position"/>
+            <command_interface name="velocity"/>
+            <command_interface name="effort"/>
+            <state_interface name="position">
+              <param name="initial_value">${initial_position}</param>
+            </state_interface>
+            <state_interface name="velocity">
+              <param name="initial_value">0.0</param>
+            </state_interface>
+            <state_interface name="effort">
+              <param name="initial_value">0.0</param>
+            </state_interface>
+          </joint>
         </xacro:unless>
       </xacro:macro>

Commit message: fix(openarm_description): make fake O6 dip joints follow on Humble too
Problem
U1: on u22/Humble, openarm_o6_bimanual.launch.py use_fake_hardware:=true
starts and the active hand joints move, but the ten *_dip joints stay at 0
(Humble full test S4: {'R_thumb_dip': (0.0, 0.279), ...}).

Root cause
In fake mode the dip joints only have state interfaces and the mock is
expected to compute them. Jazzy's mock_components reads URDF <mimic>;
Humble's only reads <param name="mimic"> / <param name="multiplier"> on the
ros2_control joint, which were not there.

Change
- openarm.bimanual.ros2_control.xacro: configure_mimic_joint takes mimic_of
  and multiplier and the fake branch adds the two params. The 20 call sites
  use the URDF values: thumb follows *_thumb_cmc_pitch (left 2.29, right
  1.86), the other fingers their *_mcp_pitch (0.89). Real branch unchanged.
- test/urdf_checks.py: new F4 - in fake mode every URDF mimic joint carries
  mimic/multiplier params equal to its URDF <mimic>, so the multipliers now
  written in two places cannot drift. G1's ros2_control summary includes
  joint params so changes to them show in the golden diff.
- test/golden.json regenerated: only the two fake bimanual o6 cases change,
  10 lines each gain params=mimic=...,multiplier=...; real cases unchanged.

Behavior change
Humble: fake O6 dips follow their parent like on Jazzy. Jazzy: unchanged
(still computed from URDF <mimic>; no warning about the params in the log).
Real hardware unchanged.

Test
Before (F4 added, old xacro): urdf_checks 167 passed, 2 failed - F4 on both
fake o6 cases (params mimic=None multiplier=None); Humble S4 FAIL (doc 10).
After xacro, before golden update: F4 passes, G1 fails only on those two
cases, as intended.
After: u24 Jazzy urdf_checks 169 passed, 0 failed, 17 known, S4 PASS,
FULL TEST PASSED. u22 Humble (run_in_docker.sh humble): D1/D2 PASS,
urdf_checks 169 passed, 0 failed, 17 known, bimanual_default S1 5 active /
S2 16 joints at 100 Hz / S3 PASS, bimanual_o6 S1-S4 PASS (36 joints at
501 Hz), H1 PASS, FULL TEST PASSED.

Docs: openarm_description/docs/11-humble-fake-mimic.md

Co-Authored-By: Claude Opus 5.5 <noreply@anthropic.com>

File: openarm_description/urdf/ros2_control/openarm.bimanual.ros2_control.xacro (robot description, xacro)
@@ -53,7 +53,9 @@
            (same as configure_joint) and is marked mimic="false": OpenArm_v10HW exports and
            drives these joints itself. Humble ignores the attribute. -->
-      <xacro:macro name="configure_mimic_joint" params="joint_name initial_position">
+      <xacro:macro name="configure_mimic_joint" params="joint_name initial_position mimic_of multiplier">
         <xacro:if value="${use_fake_hardware}">
           <joint name="${joint_name}">
+            <param name="mimic">${mimic_of}</param>
+            <param name="multiplier">${multiplier}</param>
             <state_interface name="position">
               <param name="initial_value">${initial_position}</param>
@@ -99,26 +101,26 @@
         <xacro:configure_joint joint_name="L_thumb_cmc_yaw" initial_position="0.0"/>
         <xacro:configure_joint joint_name="L_thumb_cmc_pitch" initial_position="0.0"/>
-        <xacro:configure_mimic_joint joint_name="L_thumb_dip" initial_position="0.0"/>
+        <xacro:configure_mimic_joint joint_name="L_thumb_dip" initial_position="0.0" mimic_of="L_thumb_cmc_pitch" multiplier="2.29"/>
         <xacro:configure_joint joint_name="L_index_mcp_pitch" initial_position="0.0"/>
-        <xacro:configure_mimic_joint joint_name="L_index_dip" initial_position="0.0"/>
+        <xacro:configure_mimic_joint joint_name="L_index_dip" initial_position="0.0" mimic_of="L_index_mcp_pitch" multiplier="0.89"/>
         <xacro:configure_joint joint_name="L_middle_mcp_pitch" initial_position="0.0"/>
-        <xacro:configure_mimic_joint joint_name="L_middle_dip" initial_position="0.0"/>
+        <xacro:configure_mimic_joint joint_name="L_middle_dip" initial_position="0.0" mimic_of="L_middle_mcp_pitch" multiplier="0.89"/>
         <xacro:configure_joint joint_name="L_ring_mcp_pitch" initial_position="0.0"/>
-        <xacro:configure_mimic_joint joint_name="L_ring_dip" initial_position="0.0"/>
+        <xacro:configure_mimic_joint joint_name="L_ring_dip" initial_position="0.0" mimic_of="L_ring_mcp_pitch" multiplier="0.89"/>
         <xacro:configure_joint joint_name="L_pinky_mcp_pitch" initial_position="0.0"/>
-        <xacro:configure_mimic_joint joint_name="L_pinky_dip" initial_position="0.0"/>
+        <xacro:configure_mimic_joint joint_name="L_pinky_dip" initial_position="0.0" mimic_of="L_pinky_mcp_pitch" multiplier="0.89"/>
       </xacro:if>
       <xacro:if value="${ee_type == 'o6'}">
         <xacro:configure_joint joint_name="L_thumb_cmc_yaw" initial_position="0.0"/>
         <xacro:configure_joint joint_name="L_thumb_cmc_pitch" initial_position="0.0"/>
-        <xacro:configure_mimic_joint joint_name="L_thumb_dip" initial_position="0.0"/>
+        <xacro:configure_mimic_joint joint_name="L_thumb_dip" initial_position="0.0" mimic_of="L_thumb_cmc_pitch" multiplier="2.29"/>
         <xacro:configure_joint joint_name="L_index_mcp_pitch" initial_position="0.0"/>
-        <xacro:configure_mimic_joint joint_name="L_index_dip" initial_position="0.0"/>
+        <xacro:configure_mimic_joint joint_name="L_index_dip" initial_position="0.0" mimic_of="L_index_mcp_pitch" multiplier="0.89"/>
         <xacro:configure_joint joint_name="L_middle_mcp_pitch" initial_position="0.0"/>
-        <xacro:configure_mimic_joint joint_name="L_middle_dip" initial_position="0.0"/>
+        <xacro:configure_mimic_joint joint_name="L_middle_dip" initial_position="0.0" mimic_of="L_middle_mcp_pitch" multiplier="0.89"/>
         <xacro:configure_joint joint_name="L_ring_mcp_pitch" initial_position="0.0"/>
-        <xacro:configure_mimic_joint joint_name="L_ring_dip" initial_position="0.0"/>
+        <xacro:configure_mimic_joint joint_name="L_ring_dip" initial_position="0.0" mimic_of="L_ring_mcp_pitch" multiplier="0.89"/>
         <xacro:configure_joint joint_name="L_pinky_mcp_pitch" initial_position="0.0"/>
-        <xacro:configure_mimic_joint joint_name="L_pinky_dip" initial_position="0.0"/>
+        <xacro:configure_mimic_joint joint_name="L_pinky_dip" initial_position="0.0" mimic_of="L_pinky_mcp_pitch" multiplier="0.89"/>
       </xacro:if>
     </ros2_control>
@@ -181,26 +183,26 @@
         <xacro:configure_joint joint_name="R_thumb_cmc_yaw" initial_position="0.0"/>
         <xacro:configure_joint joint_name="R_thumb_cmc_pitch" initial_position="0.0"/>
-        <xacro:configure_mimic_joint joint_name="R_thumb_dip" initial_position="0.0"/>
+        <xacro:configure_mimic_joint joint_name="R_thumb_dip" initial_position="0.0" mimic_of="R_thumb_cmc_pitch" multiplier="1.86"/>
         <xacro:configure_joint joint_name="R_index_mcp_pitch" initial_position="0.0"/>
-        <xacro:configure_mimic_joint joint_name="R_index_dip" initial_position="0.0"/>
+        <xacro:configure_mimic_joint joint_name="R_index_dip" initial_position="0.0" mimic_of="R_index_mcp_pitch" multiplier="0.89"/>
         <xacro:configure_joint joint_name="R_middle_mcp_pitch" initial_position="0.0"/>
-        <xacro:configure_mimic_joint joint_name="R_middle_dip" initial_position="0.0"/>
+        <xacro:configure_mimic_joint joint_name="R_middle_dip" initial_position="0.0" mimic_of="R_middle_mcp_pitch" multiplier="0.89"/>
         <xacro:configure_joint joint_name="R_ring_mcp_pitch" initial_position="0.0"/>
-        <xacro:configure_mimic_joint joint_name="R_ring_dip" initial_position="0.0"/>
+        <xacro:configure_mimic_joint joint_name="R_ring_dip" initial_position="0.0" mimic_of="R_ring_mcp_pitch" multiplier="0.89"/>
         <xacro:configure_joint joint_name="R_pinky_mcp_pitch" initial_position="0.0"/>
-        <xacro:configure_mimic_joint joint_name="R_pinky_dip" initial_position="0.0"/>
+        <xacro:configure_mimic_joint joint_name="R_pinky_dip" initial_position="0.0" mimic_of="R_pinky_mcp_pitch" multiplier="0.89"/>
       </xacro:if>
       <xacro:if value="${ee_type == 'o6'}">
         <xacro:configure_joint joint_name="R_thumb_cmc_yaw" initial_position="0.0"/>
         <xacro:configure_joint joint_name="R_thumb_cmc_pitch" initial_position="0.0"/>
-        <xacro:configure_mimic_joint joint_name="R_thumb_dip" initial_position="0.0"/>
+        <xacro:configure_mimic_joint joint_name="R_thumb_dip" initial_position="0.0" mimic_of="R_thumb_cmc_pitch" multiplier="1.86"/>
         <xacro:configure_joint joint_name="R_index_mcp_pitch" initial_position="0.0"/>
-        <xacro:configure_mimic_joint joint_name="R_index_dip" initial_position="0.0"/>
+        <xacro:configure_mimic_joint joint_name="R_index_dip" initial_position="0.0" mimic_of="R_index_mcp_pitch" multiplier="0.89"/>
         <xacro:configure_joint joint_name="R_middle_mcp_pitch" initial_position="0.0"/>
-        <xacro:configure_mimic_joint joint_name="R_middle_dip" initial_position="0.0"/>
+        <xacro:configure_mimic_joint joint_name="R_middle_dip" initial_position="0.0" mimic_of="R_middle_mcp_pitch" multiplier="0.89"/>
         <xacro:configure_joint joint_name="R_ring_mcp_pitch" initial_position="0.0"/>
-        <xacro:configure_mimic_joint joint_name="R_ring_dip" initial_position="0.0"/>
+        <xacro:configure_mimic_joint joint_name="R_ring_dip" initial_position="0.0" mimic_of="R_ring_mcp_pitch" multiplier="0.89"/>
         <xacro:configure_joint joint_name="R_pinky_mcp_pitch" initial_position="0.0"/>
-        <xacro:configure_mimic_joint joint_name="R_pinky_dip" initial_position="0.0"/>
+        <xacro:configure_mimic_joint joint_name="R_pinky_dip" initial_position="0.0" mimic_of="R_pinky_mcp_pitch" multiplier="0.89"/>
       </xacro:if>
     </ros2_control>
